File: hc-vitaminder-eagle/hc-vitaminder.sch (EAGLE design)
At the start: 8 parts

Commit message: updated schematic
Parts:
- added C1: 0.1nF, akstudios-adafruit:C-US025-024X044
Connections:
- net GND: now also C1.2
- net VCC: now also C1.1
Changed lines of the file:
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@@
 <part name="SW_SN" library="akstudios-adafruit" deviceset="SPST" device=""/>
 <part name="SW_OK" library="akstudios-adafruit" deviceset="SPST" device=""/>
+<part name="C1" library="akstudios-adafruit" deviceset="C-US" device="025-024X044" value="0.1nF"/>
 </parts>
 <sheets>
@@
 <attribute name="NAME" x="76.835" y="60.325" size="1.778" layer="95"/>
 <attribute name="VALUE" x="81.915" y="57.785" size="1.778" layer="96"/>
+</instance>
+<instance part="C1" gate="G$1" x="2.54" y="43.18" smashed="yes">
+<attribute name="NAME" x="3.556" y="43.815" size="1.778" layer="95"/>
+<attribute name="VALUE" x="3.556" y="38.989" size="1.778" layer="96"/>
 </instance>
 </instances>
@@
 <pinref part="SUPPLY2" gate="GND" pin="GND"/>
 <wire x1="10.16" y1="40.64" x2="10.16" y2="38.1" width="0.1524" layer="91"/>
+<pinref part="C1" gate="G$1" pin="2"/>
+<wire x1="2.54" y1="38.1" x2="10.16" y2="38.1" width="0.1524" layer="91"/>
+<junction x="10.16" y="38.1"/>
 </segment>
 </net>
@@
 <pinref part="P+3" gate="VCC" pin="VCC"/>
 <wire x1="10.16" y1="45.72" x2="10.16" y2="48.26" width="0.1524" layer="91"/>
+<pinref part="C1" gate="G$1" pin="1"/>
+<wire x1="2.54" y1="45.72" x2="10.16" y2="45.72" width="0.1524" layer="91"/>
+<junction x="10.16" y="45.72"/>
 </segment>
 </net>
